File: LEDStripBoard/LED_Driver.sch (KiCad schematic (older format))
At the start: 7 parts, among them U1 STCS2

Commit message: Add vcc Diode
Parts:
- added D3: BAT46, Diode_SMD:D_SOD-123, symbol device:D_Schottky
Connections:
- net +12V: now also D3.2 (A); no longer R5.1
- new net: D3.1 (K), R5.1
Changed lines of the file:
@@
 $Descr A4 11693 8268
 encoding utf-8
-Sheet 4 4
+Sheet 3 4
 Title ""
 Date ""
@@
 L power:+12V #PWR0108
 U 1 1 5FD1C2F1
-P 6200 2900
+P 6400 2900
 AR Path="/5FD1BD88/5FD1C2F1" Ref="#PWR0108"  Part="1"
 AR Path="/5FD2459A/5FD1C2F1" Ref="#PWR0111"  Part="1"
 AR Path="/5FD24674/5FD1C2F1" Ref="#PWR0114"  Part="1"
-F 0 "#PWR0114" H 6200 2750 50  0001 C CNN
-F 1 "+12V" H 6215 3073 50  0000 C CNN
-F 2 "" H 6200 2900 50  0001 C CNN
-F 3 "" H 6200 2900 50  0001 C CNN
-	1    6200 2900
+F 0 "#PWR0111" H 6400 2750 50  0001 C CNN
+F 1 "+12V" H 6415 3073 50  0000 C CNN
+F 2 "" H 6400 2900 50  0001 C CNN
+F 3 "" H 6400 2900 50  0001 C CNN
+	1    6400 2900
 	1    0    0    -1
 $EndComp
@@
 AR Path="/5FD2459A/5FD1CA67" Ref="U2"  Part="1"
 AR Path="/5FD24674/5FD1CA67" Ref="U3"  Part="1"
-F 0 "U3" H 5700 4250 50  0000 C CNN
+F 0 "U2" H 5700 4250 50  0000 C CNN
 F 1 "STCS2" H 6050 4250 50  0000 C CNN
 F 2 "LEDStripBoard:POWERSO-10" H 6400 3450 50  0001 C CNN
@@
 AR Path="/5FD2459A/5FD1D4DC" Ref="#PWR0112"  Part="1"
 AR Path="/5FD24674/5FD1D4DC" Ref="#PWR0115"  Part="1"
-F 0 "#PWR0115" H 5850 4450 50  0001 C CNN
+F 0 "#PWR0112" H 5850 4450 50  0001 C CNN
 F 1 "GND" H 5855 4527 50  0000 C CNN
 F 2 "" H 5850 4700 50  0001 C CNN
@@
 AR Path="/5FD2459A/5FD1E25E" Ref="R7"  Part="1"
 AR Path="/5FD24674/5FD1E25E" Ref="R10"  Part="1"
-F 0 "R10" H 5418 4396 50  0000 L CNN
+F 0 "R7" H 5418 4396 50  0000 L CNN
 F 1 "0.1" H 5418 4305 50  0000 L CNN
 F 2 "Resistor_THT:R_Axial_DIN0414_L11.9mm_D4.5mm_P20.32mm_Horizontal" V 5390 4340 50  0001 C CNN
@@
 AR Path="/5FD2459A/5FD1EDBE" Ref="R9"  Part="1"
 AR Path="/5FD24674/5FD1EDBE" Ref="R12"  Part="1"
-F 0 "R12" H 6468 3396 50  0000 L CNN
+F 0 "R9" H 6468 3396 50  0000 L CNN
 F 1 "1k" H 6468 3305 50  0000 L CNN
 F 2 "Resistor_SMD:R_0603_1608Metric_Pad1.05x0.95mm_HandSolder" V 6440 3340 50  0001 C CNN
@@
 AR Path="/5FD2459A/5FD1F40B" Ref="TP2"  Part="1"
 AR Path="/5FD24674/5FD1F40B" Ref="TP3"  Part="1"
-F 0 "TP3" V 6354 3988 50  0000 L CNN
+F 0 "TP2" V 6354 3988 50  0000 L CNN
 F 1 "TestPoint" V 6445 3988 50  0000 L CNN
 F 2 "TestPoint:TestPoint_Pad_D2.0mm" H 6600 3800 50  0001 C CNN
@@
 AR Path="/5FD2459A/5FD20498" Ref="R8"  Part="1"
 AR Path="/5FD24674/5FD20498" Ref="R11"  Part="1"
-F 0 "R11" H 5918 3196 50  0000 L CNN
+F 0 "R8" H 5918 3196 50  0000 L CNN
 F 1 "100" H 5918 3105 50  0000 L CNN
 F 2 "Resistor_SMD:R_0603_1608Metric_Pad1.05x0.95mm_HandSolder" V 5890 3140 50  0001 C CNN
@@
 AR Path="/5FD2459A/5FD20C52" Ref="C6"  Part="1"
 AR Path="/5FD24674/5FD20C52" Ref="C8"  Part="1"
-F 0 "C8" V 5198 3350 50  0000 C CNN
+F 0 "C6" V 5198 3350 50  0000 C CNN
 F 1 "0.1uF" V 5289 3350 50  0000 C CNN
 F 2 "Capacitor_SMD:C_0603_1608Metric_Pad1.05x0.95mm_HandSolder" H 5488 3200 50  0001 C CNN
@@
 Connection ~ 5850 3350
 Wire Wire Line
-	6400 3200 6400 2950
-Wire Wire Line
-	6400 2950 6200 2950
-Wire Wire Line
 	5850 2950 5850 3000
-Wire Wire Line
-	6200 2950 6200 2900
-Connection ~ 6200 2950
-Wire Wire Line
-	6200 2950 5850 2950
 $Comp
 L power:GND #PWR0110
@@
 AR Path="/5FD2459A/5FD2197A" Ref="#PWR0113"  Part="1"
 AR Path="/5FD24674/5FD2197A" Ref="#PWR0116"  Part="1"
-F 0 "#PWR0116" H 5200 3200 50  0001 C CNN
+F 0 "#PWR0113" H 5200 3200 50  0001 C CNN
 F 1 "GND" H 5205 3277 50  0000 C CNN
 F 2 "" H 5200 3450 50  0001 C CNN
@@
 AR Path="/5FD2459A/5FD21FAF" Ref="C7"  Part="1"
 AR Path="/5FD24674/5FD21FAF" Ref="C9"  Part="1"
-F 0 "C9" H 7165 4346 50  0000 L CNN
+F 0 "C7" H 7165 4346 50  0000 L CNN
 F 1 "0.47uF" H 7165 4255 50  0000 L CNN
 F 2 "Capacitor_SMD:C_0603_1608Metric_Pad1.05x0.95mm_HandSolder" H 7088 4150 50  0001 C CNN
@@
 	6250 3650 7050 3650
 Connection ~ 7050 3650
+$Comp
+L device:D_Schottky D3
+U 1 1 5FE1BEB9
+P 6100 2950
+AR Path="/5FD24674/5FE1BEB9" Ref="D3"  Part="1"
+AR Path="/5FD1BD88/5FE1BEB9" Ref="D1"  Part="1"
+AR Path="/5FD2459A/5FE1BEB9" Ref="D2"  Part="1"
+F 0 "D2" H 6100 3166 50  0000 C CNN
+F 1 "BAT46" H 6100 3075 50  0000 C CNN
+F 2 "Diode_SMD:D_SOD-123" H 6100 2950 50  0001 C CNN
+F 3 "~" H 6100 2950 50  0001 C CNN
+	1    6100 2950
+	1    0    0    -1
+$EndComp
+Wire Wire Line
+	6400 2900 6400 2950
+Wire Wire Line
+	6400 2950 6250 2950
+Connection ~ 6400 2950
+Wire Wire Line
+	6400 2950 6400 3200
+Wire Wire Line
+	5950 2950 5850 2950
 $EndSCHEMATC
